File: electrical/kicad/diy-earthroamer.kicad_sch (KiCad schematic)
At the start: 0 parts

Commit message: KiCad project: 12-symbol library, 11 hierarchical sub-sheets, 48V plan
Item 1 from the next-steps list: real KiCad project ready to draw in.

- electrical/kicad/lib/diy-earthroamer.kicad_sym: 12 custom symbols
  (Epoch 48V module, MultiPlus-II 48/5000, MPPT 250/100, Orion XS
  48-24, Cerbo GX, SmartShunt 500A, Mabru SCS 12000, Class T fuse,
  Blue Sea busbar, DC breaker, SmartPlug 30A, Linak LA36, Webasto
  Dual Top Evo 8, Garnet SeeLevel RV-C)
- electrical/kicad/sym-lib-table: registers project lib in KiCad
- 11 hierarchical sub-sheet files with valid title blocks and unique
  UUIDs: 48V_Bus, 24V_SubBus, 12V_Legacy, Solar, AC_Distribution,
  Lighting, HVAC_Control, Plumbing_Control, LiftBox_Control, Comms_AV
- diy-earthroamer.kicad_sch: root sheet now references all 11
  sub-sheets in a 4-column grid for easy navigation in KiCad
- diy-earthroamer.kicad_pro: sheets list reflects the hierarchy
- electrical/kicad/sheets/48v-bus-plan.md: detailed drawing plan for
  the first sheet — components, net names, hierarchical pins,
  step-by-step instructions with acceptance criteria
- All files validated for balanced parens

Tank vendor catalog + supplier cross-reference added to address the
'parts should come from suppliers' note:

- plumbing/tank-layout.md: RV tank vendor list (Class A Customs,
  RecPro, Icon Direct, Plastic-Mart, Ronco, PTI) with selection
  criteria for the 60-gal stock tank
- vendor-docs/suppliers.md: comprehensive supplier cross-reference
  across every subsystem so the build sources off-the-shelf where
  possible

MASTER.md now 183 KB / 4597 lines / 643 table rows.
Other:
- added sheet 12V_Legacy (sheets/12v-legacy.kicad_sch)
- added sheet 24V_SubBus (sheets/24v-subbus.kicad_sch)
- added sheet 48V_Bus (sheets/48v-bus.kicad_sch)
- added sheet AC_Distribution (sheets/ac-distro.kicad_sch)
- added sheet Comms_AV (sheets/comms-av.kicad_sch)
- added sheet HVAC_Control (sheets/hvac-control.kicad_sch)
- added sheet LiftBox_Control (sheets/liftbox.kicad_sch)
- added sheet Lighting (sheets/lighting.kicad_sch)
- added sheet Plumbing_Control (sheets/plumbing-control.kicad_sch)
- added sheet Solar (sheets/solar.kicad_sch)
Changed lines of the file:
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@@
 		(rev "0.1")
 		(company "DIY Earthroamer Project")
-		(comment 1 "Hierarchical root: see sheets-plan.md for sub-sheets")
-		(comment 2 "ABYC E-11 conventions, marine-grade harness")
-		(comment 3 "Bus voltage: 48V primary, 24V sub, 12V legacy")
-		(comment 4 "Decision basis: ADR-0004; one-line in electrical/oneline.md")
+		(comment 1 "Hierarchical root with 11 sub-sheets")
+		(comment 2 "ABYC E-11; 48V primary + 24V sub + 12V legacy")
+		(comment 3 "Symbols: project lib (lib/diy-earthroamer.kicad_sym)")
+		(comment 4 "Architecture in electrical/oneline.md and electrical/kicad/sheets-plan.md")
+	)
+	(sheet
+		(at 25.4 25.4) (size 50.8 30.48)
+		(stroke (width 0.1524) (type solid))
+		(fill (color 0 0 0 0.0000))
+		(property "Sheetname" "48V_Bus" (at 25.4 24.4 0)
+			(effects (font (size 1.524 1.524)) (justify left bottom)))
+		(property "Sheetfile" "sheets/48v-bus.kicad_sch" (at 25.4 56.5 0)
+			(effects (font (size 1.0 1.0)) (justify left top)))
+	)
+	(sheet
+		(at 88.9 25.4) (size 50.8 30.48)
+		(stroke (width 0.1524) (type solid))
+		(fill (color 0 0 0 0.0000))
+		(property "Sheetname" "24V_SubBus" (at 88.9 24.4 0)
+			(effects (font (size 1.524 1.524)) (justify left bottom)))
+		(property "Sheetfile" "sheets/24v-subbus.kicad_sch" (at 88.9 56.5 0)
+			(effects (font (size 1.0 1.0)) (justify left top)))
+	)
+	(sheet
+		(at 152.4 25.4) (size 50.8 30.48)
+		(stroke (width 0.1524) (type solid))
+		(fill (color 0 0 0 0.0000))
+		(property "Sheetname" "12V_Legacy" (at 152.4 24.4 0)
+			(effects (font (size 1.524 1.524)) (justify left bottom)))
+		(property "Sheetfile" "sheets/12v-legacy.kicad_sch" (at 152.4 56.5 0)
+			(effects (font (size 1.0 1.0)) (justify left top)))
+	)
+	(sheet
+		(at 215.9 25.4) (size 50.8 30.48)
+		(stroke (width 0.1524) (type solid))
+		(fill (color 0 0 0 0.0000))
+		(property "Sheetname" "Solar" (at 215.9 24.4 0)
+			(effects (font (size 1.524 1.524)) (justify left bottom)))
+		(property "Sheetfile" "sheets/solar.kicad_sch" (at 215.9 56.5 0)
+			(effects (font (size 1.0 1.0)) (justify left top)))
+	)
+	(sheet
+		(at 25.4 76.2) (size 50.8 30.48)
+		(stroke (width 0.1524) (type solid))
+		(fill (color 0 0 0 0.0000))
+		(property "Sheetname" "AC_Distribution" (at 25.4 75.2 0)
+			(effects (font (size 1.524 1.524)) (justify left bottom)))
+		(property "Sheetfile" "sheets/ac-distro.kicad_sch" (at 25.4 107.3 0)
+			(effects (font (size 1.0 1.0)) (justify left top)))
+	)
+	(sheet
+		(at 88.9 76.2) (size 50.8 30.48)
+		(stroke (width 0.1524) (type solid))
+		(fill (color 0 0 0 0.0000))
+		(property "Sheetname" "Lighting" (at 88.9 75.2 0)
+			(effects (font (size 1.524 1.524)) (justify left bottom)))
+		(property "Sheetfile" "sheets/lighting.kicad_sch" (at 88.9 107.3 0)
+			(effects (font (size 1.0 1.0)) (justify left top)))
+	)
+	(sheet
+		(at 152.4 76.2) (size 50.8 30.48)
+		(stroke (width 0.1524) (type solid))
+		(fill (color 0 0 0 0.0000))
+		(property "Sheetname" "HVAC_Control" (at 152.4 75.2 0)
+			(effects (font (size 1.524 1.524)) (justify left bottom)))
+		(property "Sheetfile" "sheets/hvac-control.kicad_sch" (at 152.4 107.3 0)
+			(effects (font (size 1.0 1.0)) (justify left top)))
+	)
+	(sheet
+		(at 215.9 76.2) (size 50.8 30.48)
+		(stroke (width 0.1524) (type solid))
+		(fill (color 0 0 0 0.0000))
+		(property "Sheetname" "Plumbing_Control" (at 215.9 75.2 0)
+			(effects (font (size 1.524 1.524)) (justify left bottom)))
+		(property "Sheetfile" "sheets/plumbing-control.kicad_sch" (at 215.9 107.3 0)
+			(effects (font (size 1.0 1.0)) (justify left top)))
+	)
+	(sheet
+		(at 25.4 127.0) (size 50.8 30.48)
+		(stroke (width 0.1524) (type solid))
+		(fill (color 0 0 0 0.0000))
+		(property "Sheetname" "LiftBox_Control" (at 25.4 126.0 0)
+			(effects (font (size 1.524 1.524)) (justify left bottom)))
+		(property "Sheetfile" "sheets/liftbox.kicad_sch" (at 25.4 158.1 0)
+			(effects (font (size 1.0 1.0)) (justify left top)))
+	)
+	(sheet
+		(at 88.9 127.0) (size 50.8 30.48)
+		(stroke (width 0.1524) (type solid))
+		(fill (color 0 0 0 0.0000))
+		(property "Sheetname" "Comms_AV" (at 88.9 126.0 0)
+			(effects (font (size 1.524 1.524)) (justify left bottom)))
+		(property "Sheetfile" "sheets/comms-av.kicad_sch" (at 88.9 158.1 0)
+			(effects (font (size 1.0 1.0)) (justify left top)))
 	)
 	(sheet_instances
-		(path "/"
-			(page "1")
-		)
+		(path "/" (page "1"))
 	)
 	(embedded_fonts no)
